File: KiCad files/Buggly SPD Aux.kicad_pcb (KiCad board)
At the start: 2 copper layers, 120.4 x 99.9 mm, 47 parts, among them J1 DB25_Female, J10 Screw_Terminal_01x08, J7 Screw_Terminal_01x02, J8 Screw_Terminal_01x08, J9 Screw_Terminal_01x07, K1 Panasonic_CM1-R-12V, K2 Panasonic_CM1-R-12V, Q1 AUIRF3205, Q2 AUIRF3205, Q3 AUIRF3205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

Commit message: Add files via upload
Parts:
- removed D10: LED, LED_THT:LED_D5.0mm
- removed D11: 1N4001, Diode_THT:D_DO-41_SOD81_P10.16mm_Horizontal
- D6: value 1N4001 -> LED; footprint Diode_THT:D_DO-41_SOD81_P10.16mm_Horizontal -> LED_THT:LED_D5.0mm
- moved D6 44.7 mm to (155.8, 119.3), turned to 90 degrees
- moved D5 0.67 mm to (120.2, 41.7)
- moved Q4 0.50 mm to (122.7, 38.5)
- moved R8 0.13 mm to (149.3, 103.5)
- moved RN1 0.08 mm to (151.2, 75.9)
- moved R5 0.07 mm to (155.8, 103.5)
Connections:
- net D10-control renamed D6-control
- net D10-out renamed D6-out
- net D11-control renamed D5-control
- net D11-out renamed D5-out
- net D50-control renamed D45-control
- net D52-control renamed D40-control
- net D53-control renamed D38-control
- net D53-out renamed D38-out
- D5 pad 2: F3-out -> F7-out
- D6 pad 1: D52-out -> F7-out
- D6 pad 2: F4-out -> Net-(D6-Pad2)
- J8 pad 7: D52-out -> D40-out
- Q5 pad 2: D52-out -> D40-out
- R5 pad 2: Net-(D10-Pad2) -> Net-(D6-Pad2)
- R6 pad 1: D52-out -> D40-out
Routing:
- net F7-out: track 33.6 -> 271.1 mm, vias 0 -> 1
- net F3-out: track 217.2 -> 148.5 mm, vias 5 -> 4
- net D52-out: track 52.5 -> 0.00 mm
- net D40-out: track 0.00 -> 52.5 mm, vias 0 -> 1
- net F4-out: track 151.5 -> 119.0 mm, vias 1 -> 2
- net D38-out: track 69.3 -> 62.1 mm
- net Net-(D6-Pad2): track 0.00 -> 3.10 mm
- net Net-(D10-Pad2): track 3.10 -> 0.00 mm
- net D5-out: track 124.5 -> 126.9 mm, vias 1 -> 3
- net D45-control: track 88.0 -> 86.1 mm
- net D5-control: track 104.7 -> 102.9 mm
- net 12V-Raw: track 114.1 -> 112.3 mm
- net Spare-ADC: track 19.1 -> 20.2 mm
- net GND: vias 54 -> 58
Other:
- board text added: "D38out(Ign2)"
- board text added: "D40out(Ign1)"
- board text added: "D5out(spare HC-)"
- board text added: "D6out(Idle-)"
- board text added: "SpareHC"
- board text removed: "D10out(Idle-)"
- board text removed: "D11out(spare HC-)"
- board text removed: "D52out(Ign1)"
- board text removed: "D53out(Ign2)"
- board text removed: "SprHC"
