File: KiCad files/Buggly SPD Aux.sch (KiCad schematic (older format))
At the start: 47 parts, among them J1 DB25_Female, J10 Screw_Terminal_01x08, J7 Screw_Terminal_01x02, J8 Screw_Terminal_01x08, J9 Screw_Terminal_01x07, K1 Panasonic_CM1-R-12V, K2 Panasonic_CM1-R-12V, Q1 AUIRF3205, Q2 AUIRF3205, Q3 AUIRF3205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

Commit message: Add files via upload
Parts:
- removed D10: LED, LED_THT:LED_D5.0mm, symbol V10-Ign-Inj-Drivers-V2-rescue:LED
- removed D11, D6: 1N4001, Diode_THT:D_DO-41_SOD81_P10.16mm_Horizontal, symbol Simulation_SPICE:DIODE
- added D6: LED, LED_THT:LED_D5.0mm, symbol V10-Ign-Inj-Drivers-V2-rescue:LED
Connections:
- net labels added: D38-control, D38-out, D40-control, D40-out, D45-control, D5-control, D5-out, D6-control, D6-out
- net labels removed: D10-control, D10-out, D11-control, D11-out, D50-control, D52-control, D52-out, D53-control, D53-out
- wire segments 168 -> 162
- no-connect marks 6 -> 7
Other:
- note added: "(Spare H/C out)"
- note added: "Bu"
- note added: "Dk Rd"
- note added: "Gn"
- note added: "Or"
- note added: "Rd"
- note added: "Spare H/C out"
- note added: "Yl"
- note removed: "(Spare out)"
- note removed: "Spare High Current Output -"
- note removed: "Spare high current output"
- note removed: "Spare wire"
